Commit message: feat: AR4 Physical-AI customizations
- annin_ar4_gazebo: add tabletop world with shelf + teal/magenta/yellow
  cubes as pick-and-sort targets; update gazebo.launch.py and
  CMakeLists.txt to include it; add per-model config and smolvla launch
- annin_ar4_moveit_config: fix SRDF allowed collision matrix —
  link_4_aluminum ↔ gripper_base_link overlap at the home position
  blocked all MoveIt planning; update servo + moveit launch files
- annin_ar4_description: URDF/Xacro tweaks for correct sim spawning
- annin_ar4_driver: gripper driver config update
- example_files: add COLCON_IGNORE

Co-Authored-By: Claude Sonnet 4.6 <noreply@anthropic.com>

File: annin_ar4_description/urdf/ar.urdf.xacro (robot description, xacro)
@@ -16,5 +16,5 @@
     <xacro:ar_gripper
       tf_prefix="$(arg tf_prefix)"
-      parent="$(arg tf_prefix)ee_link"
+      parent="$(arg tf_prefix)link_6"
     />
   </xacro:if>

File: annin_ar4_description/urdf/ar_gazebo.urdf.xacro (robot description, xacro)
@@ -18,5 +18,5 @@
   <xacro:ar_gripper
     tf_prefix="$(arg tf_prefix)"
-    parent="$(arg tf_prefix)ee_link"
+    parent="$(arg tf_prefix)link_6"
   />
   <xacro:ar_ros2_control
@@ -46,3 +46,27 @@
     </plugin>
   </gazebo>
+  <!-- Wrist camera sensor — Gazebo Harmonic built-in camera.
+       Image published to Gazebo topic /wrist_camera/image at 15 Hz.
+       ros_gz_bridge in gazebo.launch.py maps this to the ROS 2 topic of the same name.
+       640×480, 68.8° horizontal FOV (≈ 1.2 rad). -->
+  <gazebo reference="$(arg tf_prefix)wrist_camera_link">
+    <sensor name="wrist_camera" type="camera">
+      <always_on>true</always_on>
+      <update_rate>15</update_rate>
+      <camera>
+        <horizontal_fov>1.2</horizontal_fov>
+        <image>
+          <width>640</width>
+          <height>480</height>
+          <format>R8G8B8</format>
+        </image>
+        <clip>
+          <near>0.02</near>
+          <far>5.0</far>
+        </clip>
+      </camera>
+      <topic>/wrist_camera/image</topic>
+      <gz_frame_id>$(arg tf_prefix)wrist_camera_link</gz_frame_id>
+    </sensor>
+  </gazebo>
 </robot>

File: annin_ar4_description/urdf/ar_gripper_macro.xacro (robot description, xacro)
@@ -19,7 +19,30 @@
         </material>
       </visual>
+      <!-- Rear mounting body (Y = +0.001 to +0.019). -->
       <collision>
+        <origin xyz="0 0.010 0" rpy="0 0 0"/>
         <geometry>
-          <mesh filename="file://$(find annin_ar4_description)/meshes/ar4_gripper/gripper_base_link.stl" />
+          <box size="0.060 0.018 0.045"/>
+        </geometry>
+      </collision>
+      <!-- Palm body (Y = -0.024 to 0).  Covers the open palm mesh area that objects
+           previously clipped into silently.  At normal grasping height the palm sits
+           ~35 mm above the top of a 22 mm block, so this box never contacts objects
+           during a correct approach — it only fires if the arm descends too far.
+           Gazebo contact on this link is soft (see below) so any contact produces a
+           gentle corrective force rather than an impulse that destabilises joints 5/6. -->
+      <collision>
+        <origin xyz="0 -0.012 0" rpy="0 0 0"/>
+        <geometry>
+          <box size="0.054 0.024 0.042"/>
+        </geometry>
+      </collision>
+      <!-- Gateway lip (Y = -0.022 to -0.038): bridges the 9 mm gap between the palm
+           box and the jaw collision tops, creating a continuous barrier so objects
+           cannot slip into the palm cavity and become lodged. -->
+      <collision>
+        <origin xyz="0 -0.030 0" rpy="0 0 0"/>
+        <geometry>
+          <box size="0.040 0.016 0.034"/>
         </geometry>
       </collision>
@@ -39,7 +62,17 @@
         </material>
       </visual>
+      <!-- Main jaw body.  Inner grasping face stays at X ≈ 0 (unchanged from
+           the original 9mm box).  The body is extended OUTWARD from that face
+           to 18mm — doubling the wall thickness so a block flung by a corner
+           contact cannot tunnel through in a single physics step.  This mirrors
+           the plank collision strategy (thick box, solid geometry).
+           Jaw Y shortened from 0.032 to 0.028 (nose pulled back 4 mm): the
+           catch-ledge at the jaw tip is smaller, so a slightly rotated block
+           corner is less likely to wedge.  Gateway-lip overlap increases from
+           5.5 mm to 13.5 mm so no gap opens at the back of the jaw. -->
       <collision>
+        <origin xyz="-0.00914 -0.0115 -0.0013" rpy="0 0 0"/>
         <geometry>
-          <mesh filename="file://$(find annin_ar4_description)/meshes/ar4_gripper/gripper_jaw1_link.stl" />
+          <box size="0.018 0.028 0.034"/>
         </geometry>
       </collision>
@@ -59,7 +92,12 @@
         </material>
       </visual>
+      <!-- Main jaw body — mirrors jaw1.  Inner face stays at base-frame X ≈ 0;
+           extended outward (local -X direction, which is base +X due to the
+           π-around-Y rotation) to 18mm for anti-tunneling.
+           Y shortened to 0.028 to match jaw1 nose-length reduction. -->
       <collision>
+        <origin xyz="-0.00874 -0.0115 0.0001" rpy="0 0 0"/>
         <geometry>
-          <mesh filename="file://$(find annin_ar4_description)/meshes/ar4_gripper/gripper_jaw2_link.stl" />
+          <box size="0.018 0.028 0.032"/>
         </geometry>
       </collision>
@@ -85,4 +123,38 @@
       <mimic joint="${tf_prefix}gripper_jaw1_joint" multiplier="1" offset="0"/>
     </joint>
+    <!-- Soft, nearly frictionless contact on the gripper base: kp=5000 keeps corrective
+         forces gentle; mu≈0 means objects that touch the palm/lip slide away rather
+         than sticking and becoming lodged. -->
+    <gazebo reference="${tf_prefix}gripper_base_link">
+      <mu1>0.05</mu1>
+      <mu2>0.05</mu2>
+      <kp>5000</kp>
+      <kd>100</kd>
+      <maxVel>0.3</maxVel>
+      <minDepth>0.003</minDepth>
+    </gazebo>
+    <!-- High friction on jaw surfaces so objects don't slip or ragdoll on contact.
+         kp/kd matched to block surfaces (100000/50) so the combined ODE stiffness
+         is symmetric — asymmetric stiffness causes contact-induced rotation.
+         kp lowered from 200000 to 100000: combined stiffness is 50000 N/m, still
+         firm (50 N at 1 mm penetration, 150 N friction per jaw >> 0.3 N gravity),
+         but peak contact impulses are halved, keeping the kinematic chain stable.
+         mu raised to 3.0 (rubber-tipped jaws) to compensate for the lower kp. -->
+    <gazebo reference="${tf_prefix}gripper_jaw1_link">
+      <mu1>3.0</mu1>
+      <mu2>3.0</mu2>
+      <kp>100000</kp>
+      <kd>50</kd>
+      <maxVel>0.01</maxVel>
+      <minDepth>0.001</minDepth>
+    </gazebo>
+    <gazebo reference="${tf_prefix}gripper_jaw2_link">
+      <mu1>3.0</mu1>
+      <mu2>3.0</mu2>
+      <kp>100000</kp>
+      <kd>50</kd>
+      <maxVel>0.01</maxVel>
+      <minDepth>0.001</minDepth>
+    </gazebo>
   </xacro:macro>
 </robot>

File: annin_ar4_description/urdf/ar_macro.xacro (robot description, xacro)
@@ -458,4 +458,5 @@
          effort="-1"
          velocity="1.0472"/>
+  <dynamics damping="0.5" friction="0.0"/>
 </joint>
 <!-- ===================== -->
@@ -503,11 +504,37 @@
     effort="-1"
     velocity="1.5708"/>
-</joint>
-    <!-- center of the end effector mounting surface on link_6 -->
+  <dynamics damping="0.5" friction="0.0"/>
+</joint>
+    <!-- ee_link is the MoveIt/Servo TCP — placed at the jaw tips so Cartesian commands
+         land the gripper opening at the target, not the wrist flange.
+         Offset derived from jaw mesh geometry: jaw tips sit 64 mm along link_6 +Z
+         (the approach axis).  The gripper is parented directly to link_6 (not ee_link)
+         so the physical gripper mesh stays at the correct wrist position. -->
     <link name="${tf_prefix}ee_link" />
     <joint name="${tf_prefix}ee_joint" type="fixed">
       <parent link="${tf_prefix}link_6" />
       <child link="${tf_prefix}ee_link" />
-      <origin xyz="0 0 0" rpy="0 0 0" />
+      <origin xyz="0 0 0.064" rpy="0 0 0" />
+    </joint>
+    <!-- Wrist camera: top-mounted on gripper_base_link.
+         gripper_base_link axes (relative to ee_link, joint Rx(-90°)):
+           +X = jaw opening axis (left-right)
+           +Y = backward along tool (toward wrist)   ← gripper_base -Y = link_6 +Z = toward object
+           +Z = dorsal/top face of the gripper palm  ← where this camera sits
+         xyz="0 0 0.04": 4 cm in gripper_base +Z = on the top surface of the palm.
+         rpy="0 0 -1.5708": Rz(-90°) rotates camera so its +X (gz-sim optical axis)
+         aligns with gripper_base -Y = link_6 +Z = the approach/tool axis.
+         The camera therefore looks straight toward the jaws and the object. -->
+    <link name="${tf_prefix}wrist_camera_link">
+      <inertial>
+        <mass value="0.001"/>
+        <origin xyz="0 0 0" rpy="0 0 0"/>
+        <inertia ixx="1e-6" ixy="0" ixz="0" iyy="1e-6" iyz="0" izz="1e-6"/>
+      </inertial>
+    </link>
+    <joint name="${tf_prefix}wrist_camera_joint" type="fixed">
+      <parent link="${tf_prefix}gripper_base_link"/>
+      <child link="${tf_prefix}wrist_camera_link"/>
+      <origin xyz="0 0 0.04" rpy="0 0 -1.5708"/>
     </joint>
   </xacro:macro>

File: annin_ar4_moveit_config/srdf/ar_macro.srdf.xacro (robot description, xacro)
@@ -54,4 +54,8 @@
     <disable_collisions link1="${tf_prefix}link_6_aluminum" link2="${tf_prefix}gripper_base_link" reason="Adjacent" />
     <disable_collisions link1="${tf_prefix}link_5_aluminum" link2="${tf_prefix}gripper_base_link" reason="Adjacent" />
+    <!-- At the all-zeros home position the gripper folds back far enough that
+         link_4_aluminum and gripper_base_link overlap in collision space.
+         Disable this pair so planning is not blocked at startup. -->
+    <disable_collisions link1="${tf_prefix}link_4_aluminum" link2="${tf_prefix}gripper_base_link" reason="Default" />
   </xacro:macro>
 </robot>
