Commit message: feat(sim): replace wrist camera with static top camera, match real rig views
The physical rig observes the arm with two fixed cameras (side/scene + high-
oblique top) and has no wrist camera, so the sim now matches:

- Remove the gripper-mounted wrist_camera link/joint and its Gazebo sensor
  from the URDF; cameras are now world models only.
- Add a static top_camera model to both tabletop worlds, publishing
  /top_camera/image (bridged like scene_camera).
- Re-aim scene_camera to the real C920's vantage: just above table height,
  ~0.9 m out, near-horizontal.
- Camera poses tuned by 50% overlay of sim frames against the rig's pinned
  reference frames with the arm at HOME [0,-0.3,0.5,0,1.2,0]; arm, plank,
  and objects line up in both views. Reference frames live in the main repo
  under data/camera_reference/2026-08-30/.
- Add a far_wall (-Y) backdrop, the wall the side camera actually sees,
  and move back_wall outward so it clears the pulled-back side camera.
- Rename bridge.yaml mappings /wrist_camera/* -> /top_camera/*.

Co-Authored-By: Claude Fable 5 <noreply@anthropic.com>
Claude-Session: https://claude.ai/code/session_01TMDbss3mbMdoTEoFyBekSP

File: annin_ar4_description/urdf/ar_gazebo.urdf.xacro (robot description, xacro)
@@ -46,27 +46,8 @@
     </plugin>
   </gazebo>
-  <!-- Wrist camera sensor — Gazebo Harmonic built-in camera.
-       Image published to Gazebo topic /wrist_camera/image at 15 Hz.
-       ros_gz_bridge in gazebo.launch.py maps this to the ROS 2 topic of the same name.
-       640×480, 68.8° horizontal FOV (≈ 1.2 rad). -->
-  <gazebo reference="$(arg tf_prefix)wrist_camera_link">
-    <sensor name="wrist_camera" type="camera">
-      <always_on>true</always_on>
-      <update_rate>15</update_rate>
-      <camera>
-        <horizontal_fov>1.2</horizontal_fov>
-        <image>
-          <width>640</width>
-          <height>480</height>
-          <format>R8G8B8</format>
-        </image>
-        <clip>
-          <near>0.02</near>
-          <far>5.0</far>
-        </clip>
-      </camera>
-      <topic>/wrist_camera/image</topic>
-      <gz_frame_id>$(arg tf_prefix)wrist_camera_link</gz_frame_id>
-    </sensor>
-  </gazebo>
+  <!-- No robot-mounted cameras. The physical rig observes the arm with two static
+       cameras (side/scene + top, both off-arm), so the sim cameras are static
+       models in the world SDF (scene_camera + top_camera in the tabletop worlds),
+       not URDF sensors. A wrist camera used to live here — removed when the rig
+       decision landed on side+top with no wrist cam. -->
 </robot>

File: annin_ar4_description/urdf/ar_macro.xacro (robot description, xacro)
@@ -517,25 +517,4 @@
       <origin xyz="0 0 0.064" rpy="0 0 0" />
     </joint>
-    <!-- Wrist camera: top-mounted on gripper_base_link.
-         gripper_base_link axes (relative to ee_link, joint Rx(-90°)):
-           +X = jaw opening axis (left-right)
-           +Y = backward along tool (toward wrist)   ← gripper_base -Y = link_6 +Z = toward object
-           +Z = dorsal/top face of the gripper palm  ← where this camera sits
-         xyz="0 0 0.04": 4 cm in gripper_base +Z = on the top surface of the palm.
-         rpy="0 0 -1.5708": Rz(-90°) rotates camera so its +X (gz-sim optical axis)
-         aligns with gripper_base -Y = link_6 +Z = the approach/tool axis.
-         The camera therefore looks straight toward the jaws and the object. -->
-    <link name="${tf_prefix}wrist_camera_link">
-      <inertial>
-        <mass value="0.001"/>
-        <origin xyz="0 0 0" rpy="0 0 0"/>
-        <inertia ixx="1e-6" ixy="0" ixz="0" iyy="1e-6" iyz="0" izz="1e-6"/>
-      </inertial>
-    </link>
-    <joint name="${tf_prefix}wrist_camera_joint" type="fixed">
-      <parent link="${tf_prefix}gripper_base_link"/>
-      <child link="${tf_prefix}wrist_camera_link"/>
-      <origin xyz="0 0 0.04" rpy="0 0 -1.5708"/>
-    </joint>
   </xacro:macro>
 </robot>
