Commit message: fix(sim): 20 N jaw effort limit so a full close grasps stably
The recorder commands a full close (AURA-811). With effort=-1 and 1000 on
the position-controlled jaws, Gazebo drove them 10-13 mm into the object
and the contact solve shoved or ejected it; about half the grasps missed.
A 20 N limit on both jaws gave 23/24 grasps across all six objects in
the spice-rack world; 10 N barely closed the jaws and 40 N was unstable.
Only Gazebo reads this limit; the servo hardware interface ignores it.

Co-Authored-By: Claude Opus 5 (1M context) <noreply@anthropic.com>
Claude-Session: https://claude.ai/code/session_01EWgyTCGSRt9YnXvaFhg87j

File: annin_ar4_description/urdf/ar_gripper_macro.xacro (robot description, xacro)
@@ -108,4 +108,11 @@
       </inertial>
     </link>
+    <!-- Jaw effort limit (both jaws): 20 N. Only Gazebo uses it; the servo hardware
+         interface ignores <limit effort>. With the recorder's full close (AURA-811),
+         unlimited effort drove the position-controlled jaws 10-13 mm into the object
+         and the contact solve shoved or ejected it: about half the grasps missed. 20 N
+         gave 23/24 grasps across all six objects on 2026-09-13; 10 N barely closed the
+         jaws and 40 N was unstable again. The real HPS-3518SG gripper squeezes an
+         estimated 50-75 N per jaw, so this is a stability setting, not a force match. -->
     <joint name="${tf_prefix}gripper_jaw1_joint" type="prismatic">
       <origin xyz="0.0 -0.036 0" rpy="0.0 0.0 0.0"/>
@@ -113,5 +120,5 @@
       <child link="${tf_prefix}gripper_jaw1_link"/>
       <axis xyz="-1 0 0"/>
-      <limit lower="0" upper="0.014" effort="-1" velocity="1.0"/>
+      <limit lower="0" upper="0.014" effort="20" velocity="1.0"/>
     </joint>
     <joint name="${tf_prefix}gripper_jaw2_joint" type="prismatic">
@@ -120,5 +127,5 @@
       <child link="${tf_prefix}gripper_jaw2_link"/>
       <axis xyz="-1 0 0"/>
-      <limit lower="0" upper="0.014" effort="1000" velocity="1.0"/>
+      <limit lower="0" upper="0.014" effort="20" velocity="1.0"/>
       <mimic joint="${tf_prefix}gripper_jaw1_joint" multiplier="1" offset="0"/>
     </joint>
